File: PCB/snips_controller.kicad_pcb (KiCad board)
At the start: 4 copper layers, 35 x 99.9 mm, 95 parts

Commit message: Port Snips controller hardware design to Stackup (#62)
Replace the KiCad schematics with a KDL electrical design backed by the
pinned Stackup parts library. Keep the routed KiCad PCB and add Stackup
identities so the plugin can sync design changes without rerouting. Export
purchasing data with stackup bom, including hand-installed parts.

Add a Cargo-locked Stackup CLI and GitHub Actions checks for the design,
purchasing BOM, and read-only PCB sync. CI also runs the native tests and
ESP32-S3 firmware build.
Parts:
- BT1: value PH 2-pin battery RIGHT-ANGLE HORIZONTAL | S2B-PH-K(LF)(SN) | JST | THT right-angle horizontal 2.00mm -> PH 2-pin battery RIGHT-ANGLE HORIZONTAL
- C_3V3_1, C_XBEE_VCC4: value 10µF | CL10A106KP8NNNC | Samsung Electro-Mechanics | 0603 -> 10µF
- C_3V3_2, C_DBNC1, C_HALL1, C_LATCH_G1, C_OLED_2, C_RGB1, C_STICK1, C_SYS_2, C_VIN_2, C_XBEE_RC1, C_XBEE_VCC1: value 100nF | CL05B104KO5NNNC | Samsung Electro-Mechanics | 0402 -> 100nF
- C_3V3_3: value 39pF | CC0402JRNPO9BN390 | Yageo | 0402 -> 39pF
- C_ACCEL_1: value 10nF | CL05B103KB5NNNC | Samsung Electro-Mechanics | 0402 -> 10nF
- C_ACCEL_2: value 100pF | 0402CG101J500NT | FH (Guangdong Fenghua Advanced Tech) | 0402 -> 100pF
- C_ACCEL_3: value 2.2nF | CL05B222KB5NNNC | Samsung Electro-Mechanics | 0402 -> 2.2nF
- C_BAT1, C_BUCK_IN1, C_OLED_1, C_SYS_1, C_VIN_1: value 10µF | CL21A106KAYNNNE | Samsung Electro-Mechanics | 0805 -> 10µF
- C_BUCK_OUT1: value 22µF | CL21A226MAQNNNE | Samsung Electro-Mechanics | 0805 -> 22µF
- C_XBEE_VCC2: value 1µF | CL10A105KB8NNNC | Samsung Electro-Mechanics | 0603 -> 1µF
- C_XBEE_VCC3: value 47pF | 0402CG470J500NT | FH (Guangdong Fenghua Advanced Tech) | 0402 -> 47pF
- D_INV_ISO1: value BAT54W-7-F | Diodes Incorporated | SOT-323 (SC-70) -> BAT54W-7-F
- D_OR1, D_OR2: value 1N4148W | ST(Semtech) | SOD-123 -> 1N4148W
- D_RGB1: value SK6812MINI-E-012 | SK6812MINI-E | OPSCO Optoelectronics | SMD 3.2x2.8mm -> SK6812MINI-E-012
- D_VBUS_TVS1: value TPPESD5V0S1BA | TECH PUBLIC | SOD-323 -> TPPESD5V0S1BA
- J_USB1: value USB-C | TYPE-C-31-M-12 | Hroparts Elec | USB-C receptacle -> USB-C
- L_BUCK1: value 2.2µH | SRN4018-2R2M | Bourns | 4.0x4.0mm SMD -> 2.2µH
- Q_INV1: value MMBT3904(RANGE:100-300) | Jiangsu Changjing Electronics Technology Co Ltd | SOT-23 -> MMBT3904(RANGE:100-300)
- Q_LATCH1: value AO3400A | Alpha & Omega Semicon | SOT-23 -> AO3400A
- Q_PWR1: value AO3401A | Alpha & Omega Semicon | SOT-23 -> AO3401A
- R_BOOT_PU1, R_EN_PU1, R_STAT1, R_STAT2, R_TS1, R_XBEE_ATTN_PU1, R_XBEE_RST1: value 10kΩ | 0402WGF1002TCE | UNI-ROYAL(Uniroyal Elec) | 0402 -> 10kΩ
- R_BTN_PU1, R_GATE1, R_INV_BASE1, R_INV_PU1, R_PWR_EN_PD1, R_VSYS2: value 100kΩ | 0402WGF1003TCE | UNI-ROYAL(Uniroyal Elec) | 0402 -> 100kΩ
- R_CC1, R_CC2: value 5.1kΩ | 0402WGF5101TCE | UNI-ROYAL(Uniroyal Elec) | 0402 -> 5.1kΩ
- R_FB1: value RC0402FR-07255KL | Yageo | 0402 -> 255kΩ
- R_FB2: value 56.2kΩ | RC0402FR-0756K2L | Yageo | 0402 -> 56.2kΩ
- R_ISET1: value AC0402FR-07604RL | Yageo | 0402 -> 604Ω
- R_LATCH_G1: value 1MΩ | 0402WGF1004TCE | UNI-ROYAL(Uniroyal Elec) | 0402 -> 1MΩ
- R_RGB1: value 0402WGF4700TCE | UNI-ROYAL(Uniroyal Elec) | 0402 -> 470Ω
- R_USB_DM1, R_USB_DP1: value RC0402FR-0727RL | Yageo | 0402 -> 27Ω
- R_VSET1: value RC0402FR-0718KL | Yageo | 0402 -> 18kΩ
- R_VSYS1: value 200kΩ | 0402WGF2003TCE | UNI-ROYAL(Uniroyal Elec) | 0402 -> 200kΩ
- R_XBEE_RC1: value 0402WGF1000TCE | UNI-ROYAL(Uniroyal Elec) | 0402 -> 100Ω
- SW_BOOT1: value Panasonic_EVQP2 | EVQP2T02M | Panasonic | SMD tactile 2.1mm -> Panasonic_EVQP2
- SW_MACRO1, SW_MACRO2, SW_MACRO3, SW_MACRO4, SW_MACRO5, SW_MACRO6: value 6x6x5mm SMD Tactile | 1TS009A-1800-5000-CT | Hongyuan Precision | SMD tactile 6x6x5mm -> 6x6x5mm SMD Tactile
- SW_PWR1, SW_THR_DN1, SW_THR_UP1, SW_TRIG_DIG1, SW_VOL_DN1, SW_VOL_UP1: value SKRTLAE010 | Alps Alpine | SMD tactile horizontal -> SKRTLAE010
- U_ACCEL1: value QMA6100P | QST | LGA-12 2x2mm -> QMA6100P
- U_BUCK1: value TLV62569DBVR | Texas Instruments | SOT-23-5 -> TLV62569DBVR
- U_CHG1: value BQ25185DLHR | Texas Instruments | WSON-10 2.2x2.0mm -> BQ25185DLHR
- U_HALL1: value DRV5055A2QLPGM | Texas Instruments | TO-92 THT -> DRV5055A2QLPGM
- U_MCU1: value ESP32-S3-WROOM-1-N8 | Espressif Systems | SMD module 18x25.5mm -> ESP32-S3-WROOM-1-N8
- U_OLED1: value JST-SH_4Pin_OLED | SM04B-SRSS-TB(LF)(SN) | JST | SMD horizontal 1.00mm 4-pin -> Qwiic connector
- U_XBEE1: value XBee3 | XB3-24Z8UT-J | Digi International | XBee through-hole -> XBee3
- renumbered REF** to FID1, REF** to FID2, REF** to FID3, REF** to FID4, REF** to FID5, REF** to FID6, G*** to LOGO1, G*** to LOGO2, G*** to LOGO3, MHole to MH1, MHole to MH2, MHole to MH3, MHole to MH4
Connections:
- D_INV_ISO1 pad 2: unconnected-(D_INV_ISO1-NC-Pad2) -> (no net)
- D_RGB1 pad 4: unconnected-(D_RGB1-DOUT-Pad4) -> (no net)
- J_USB1 pad A8: unconnected-(J_USB1-SBU1-PadA8) -> (no net)
- J_USB1 pad B8: unconnected-(J_USB1-SBU2-PadB8) -> (no net)
- U_ACCEL1 pad 6: unconnected-(U_ACCEL1-INT2-Pad6) -> (no net)
- U_ACCEL1 pad 7: unconnected-(U_ACCEL1-NC-Pad7) -> (no net)
- U_CHG1 pad 12: (no net) -> GND
- U_CHG1 pad 13: (no net) -> GND
- U_MCU1 pad 15: unconnected-(U_MCU1-GPIO3/TOUCH3/ADC1_CH2-Pad15) -> (no net)
- U_MCU1 pad 26: unconnected-(U_MCU1-GPIO45-Pad26) -> (no net)
- U_XBEE1 pad 12: unconnected-(U_XBEE1-~{CTS}/DIO7-Pad12) -> (no net)
- U_XBEE1 pad 14: unconnected-(U_XBEE1-[RESERVED]_2-Pad14) -> (no net)
- U_XBEE1 pad 15: unconnected-(U_XBEE1-ASSOCIATE/DIO5-Pad15) -> (no net)
- U_XBEE1 pad 16: unconnected-(U_XBEE1-~{RTS}/DIO6-Pad16) -> (no net)
- U_XBEE1 pad 2: unconnected-(U_XBEE1-DOUT/DIO13-Pad2) -> (no net)
- U_XBEE1 pad 20: unconnected-(U_XBEE1-AD0_/DIO0-Pad20) -> (no net)
- U_XBEE1 pad 3: unconnected-(U_XBEE1-DIN/~{CONFIG}/DIO14-Pad3) -> (no net)
- U_XBEE1 pad 6: unconnected-(U_XBEE1-RSSI_PWM/DIO10-Pad6) -> (no net)
- U_XBEE1 pad 7: unconnected-(U_XBEE1-PWM1/DIO11-Pad7) -> (no net)
- U_XBEE1 pad 8: unconnected-(U_XBEE1-[RESERVED]_1-Pad8) -> (no net)
