File: PCB/snips_controller.kicad_pcb (KiCad board)
At the start: 4 copper layers, 35 x 99.9 mm, 95 parts

Commit message: fix: replace reverse-mount SK6812MINI-E with top-mount SK6812MINI-HS
D_RGB1 is mounted lens-up, but the SK6812MINI-E footprint used the
datasheet's bottom-view land pattern (correct only for lens-down reverse
mounting) and had no body cutout. Mounted lens-up, every pin landed on the
wrong net and no rotation could fix it, and the part's mid-body leads
could not reach the pads on a flat board.

Switch to the OPSCO SK6812MINI-HS (LCSC C2922787), a flat-bottom 3535
top-mount part with the same pins and protocol:

- New SnipsControllers_Custom:SK6812MINI-HS-012 footprint from datasheet
  Rev B/0 section 6 (top view). Pad numbers are the datasheet pin numbers:
  1 GND (chamfered corner, marked), 2 DIN, 3 VDD, 4 DOUT.
- Local sk6812mini-hs Stackup part; D_RGB1 placement and purchasing updated.
- PCB synced from Stackup and LED re-routed; production files regenerated.
- Remove the unused MINI-E footprint and the mislabeled 5050 SK6812
  datasheet; add the MINI-HS datasheet.

Co-Authored-By: Claude Opus 5.5 <noreply@anthropic.com>
Parts:
- D_RGB1: value SK6812MINI-E-012 -> SK6812MINI-HS-012; footprint SnipsControllers_Custom:SK6812MINI-E-012 -> SK6812MINI-HS-012
Routing:
- net 3V3: track 66.4 -> 71.7 mm
- net /RGB_LED/RGB_DIN_R: track 4.94 -> 2.51 mm
- net GND: track 176.2 -> 178.4 mm
